Commit message: underwater 0.0

File: ECA_A9_AUV/configuration/robots/eca_a9_default.urdf.xacro (robot description, xacro)
@@ -17,5 +17,5 @@
   <xacro:arg name="inertial_reference_frame" default="world"/>
   <!-- Include the UUV macro file -->
-  <xacro:include filename="$(find eca_a9_description)/urdf/eca_a9_base.xacro"/>
+  <xacro:include filename="$(find configuration)/urdf/eca_a9_base.xacro"/>
   <!-- Create the eca_a9 -->
   <xacro:eca_a9_base

File: ECA_A9_AUV/configuration/urdf/eca_a9_base.xacro (robot description, xacro)
@@ -14,8 +14,8 @@
 <robot xmlns:xacro="http://www.ros.org/wiki/xacro" >
   <!-- Import macro files -->
-  <xacro:include filename="$(find uuv_descriptions)/urdf/common.urdf.xacro" />
-  <xacro:include filename="$(find uuv_sensor_ros_plugins)/urdf/sensor_snippets.xacro"/>
+  <xacro:include filename="$(find tools)/urdf/common.urdf.xacro" />
+  <!--xacro:include filename="$(find uuv_sensor_ros_plugins)/urdf/sensor_snippets.xacro"/>
   <xacro:include filename="$(find eca_a9_description)/urdf/eca_a9_snippets.xacro"/>
-  <xacro:include filename="$(find uuv_gazebo_ros_plugins)/urdf/snippets.xacro"/>
+  <xacro:include filename="$(find uuv_gazebo_ros_plugins)/urdf/snippets.xacro"/>-->
   <!-- Properties -->
   <xacro:property name="mass" value="69.7"/>
@@ -28,8 +28,8 @@
   <xacro:property name="area" value="0.04155"/>
   <xacro:property name="length" value="1.98"/>
-  <xacro:property name="visual_mesh_file" value="file://$(find eca_a9_description)/mesh/eca_a9.dae"/>
-  <xacro:property name="collision_mesh_file" value="file://$(find eca_a9_description)/mesh/eca_a9.stl"/>
-  <xacro:property name="prop_mesh_file" value="file://$(find eca_a9_description)/mesh/eca_a9_propeller.dae"/>
-  <xacro:property name="fin_mesh_file" value="file://$(find eca_a9_description)/mesh/eca_a9_fin.dae"/>
+  <xacro:property name="visual_mesh_file" value="file://$(find configuration)/mesh/eca_a9.dae"/>
+  <xacro:property name="collision_mesh_file" value="file://$(find configuration)/mesh/eca_a9.stl"/>
+  <xacro:property name="prop_mesh_file" value="file://$(find configuration)/mesh/eca_a9_propeller.dae"/>
+  <xacro:property name="fin_mesh_file" value="file://$(find configuration)/mesh/eca_a9_fin.dae"/>
   <xacro:macro name="eca_a9_base" params="namespace debug inertial_reference_frame">
     <link name="${namespace}/base_link">
@@ -56,5 +56,5 @@
     <!-- Set up hydrodynamic plugin -->
     <gazebo>
-      <plugin name="${namespace}_uuv_plugin" filename="libuuv_underwater_object_ros_plugin.so">
+      <plugin name="${namespace}plugin" filename="libunderwater_object_ros_plugin.so">
         <fluid_density>${rho}</fluid_density>
         <flow_velocity_topic>hydrodynamics/current_velocity</flow_velocity_topic>
@@ -108,5 +108,5 @@
     </xacro:thruster_module_first_order_basic_fcn_macro>
     <!-- TODO: Parametrize the battery unit -->
-    <xacro:basic_linear_battery_macro
+    <!--xacro:basic_linear_battery_macro
       namespace="${namespace}"
       parent_link="${namespace}/base_link"
@@ -119,6 +119,6 @@
       smooth_current_tau="1.9499"
       voltage="4.2"
-      update_rate="2.0"/>
-    <xacro:include filename="$(find eca_a9_description)/urdf/eca_a9_sensors.xacro"/>
+      update_rate="2.0"/>-->
+    <!--xacro:include filename="$(find configuration)/urdf/eca_a9_sensors.xacro"/>-->
   </xacro:macro>
 </robot>
